File: schema/Groupe7.brd (EAGLE design)
At the start: 100 x 80 mm, 21 parts, among them T1 2N2222, T2 2N2222

Commit message: final .brd
Parts:
- added R13, R14: (no value), rcl:0207/7
- moved T1 30.0 mm to (30.5, 8.89)
- moved R10 23.7 mm to (57.1, 38.1), turned to 0 degrees
- moved R11 21.0 mm to (14.0, 20.3), turned to 270 degrees
- moved T2 18.9 mm to (30.5, 17.8)
- moved LED1 16.1 mm to (7.62, 6.35)
- moved LED2 13.7 mm to (21.6, 6.35)
- moved R12 13.3 mm to (20.3, 20.3), turned to 270 degrees
- moved DIS2 8.52 mm to (87.6, 52.1)
- moved DIS1 8.03 mm to (72.4, 52.1)
- moved R1 7.73 mm to (5.08, 20.3)
- moved IC1 6.35 mm to (41.9, 45.7)
- moved R8 4.02 mm to (57.1, 64.8)
- moved R3 4.02 mm to (57.1, 41.9)
- moved R4 4.02 mm to (57.1, 45.7)
- moved R7 4.02 mm to (57.1, 57.1)
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Connections:
- new net N$37: R13.2, R14.1, U$1.31
- net N$22: now also R13.1; no longer U$1.31
- net N$23: now also R14.2
Routing:
- net N$37: track 0.00 -> 143.6 mm
- net N$19: track 157.1 -> 286.2 mm
- net N$15: track 130.9 -> 37.5 mm
- net N$23: track 79.5 -> 172.3 mm
- net N$21: track 79.8 -> 7.32 mm
- net N$16: track 109.0 -> 44.9 mm
- net N$22: track 69.1 -> 8.78 mm
- net N$25: track 69.8 -> 116.6 mm
- net N$24: track 130.9 -> 99.1 mm
- net N$14: track 55.0 -> 36.0 mm
- net N$26: track 3.81 -> 22.4 mm
- net N$13: track 39.6 -> 25.0 mm
- net N$30: track 3.65 -> 13.9 mm
- net N$2: track 7.98 -> 17.5 mm
- net N$32: track 6.47 -> 15.8 mm
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- removed copper zone on layer 16, net GND
Other:
- board text removed: "GROUPE 7"
