File: schema/Groupe7.sch (EAGLE design)
At the start: 19 parts, among them T1 2N2222, T2 2N2222

Commit message: final .brd
Parts:
- added R11, R12, R13, R14: (no value), rcl:R-EU_0207/7
- R1, R10, R2, R3, R4, R5, R6, R7, R8, R9: device rcl:R-EU_0204/2V -> rcl:R-EU_0207/7
Connections:
- new net N$35: R11.2, T1.B
- new net N$36: R12.2, T2.B
- new net N$37: R13.2, R14.1, U$1.31
- net N$22: now also R13.1; no longer U$1.31
- net N$23: now also R14.2
- net N$28: now also R12.1; no longer T2.B
- net N$30: now also R11.1; no longer T1.B
Changed lines of the file:
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@@
 <settings>
 <setting alwaysvectorfont="no"/>
+<setting keepoldvectorfont="yes"/>
 <setting verticaltext="up"/>
 </settings>
@@
 </classes>
 <parts>
-<part name="JP1" library="pinhead" library_urn="urn:adsk.eagle:library:325" deviceset="PINHD-1X4" device="" package3d_urn="urn:adsk.eagle:package:22407/2"/>
+<part name="JP1" library="pinhead" deviceset="PINHD-1X4" device=""/>
 <part name="U$1" library="pipico" deviceset="RASPBERRY-PI-PICO_TH" device=""/>
-<part name="LED1" library="led" library_urn="urn:adsk.eagle:library:259" deviceset="LED" device="5MM" package3d_urn="urn:adsk.eagle:package:15799/2"/>
-<part name="R1" library="rcl" library_urn="urn:adsk.eagle:library:334" deviceset="R-EU_" device="0204/2V" package3d_urn="urn:adsk.eagle:package:23495/1"/>
-<part name="T1" library="transistor" library_urn="urn:adsk.eagle:library:402" deviceset="2N2222" device="" package3d_urn="urn:adsk.eagle:package:28526/2"/>
-<part name="DIS1" library="display-hp" library_urn="urn:adsk.eagle:library:212" deviceset="HD-H103" device="" package3d_urn="urn:adsk.eagle:package:13006/1"/>
-<part name="DIS2" library="display-hp" library_urn="urn:adsk.eagle:library:212" deviceset="HD-H103" device="" package3d_urn="urn:adsk.eagle:package:13006/1"/>
-<part name="IC1" library="ic-package" library_urn="urn:adsk.eagle:library:239" deviceset="DIL16" device="" package3d_urn="urn:adsk.eagle:package:922/2"/>
-<part name="LED2" library="led" library_urn="urn:adsk.eagle:library:259" deviceset="LED" device="5MM" package3d_urn="urn:adsk.eagle:package:15799/2"/>
-<part name="R2" library="rcl" library_urn="urn:adsk.eagle:library:334" deviceset="R-EU_" device="0204/2V" package3d_urn="urn:adsk.eagle:package:23495/1"/>
-<part name="R3" library="rcl" library_urn="urn:adsk.eagle:library:334" deviceset="R-EU_" device="0204/2V" package3d_urn="urn:adsk.eagle:package:23495/1"/>
-<part name="R4" library="rcl" library_urn="urn:adsk.eagle:library:334" deviceset="R-EU_" device="0204/2V" package3d_urn="urn:adsk.eagle:package:23495/1"/>
-<part name="R5" library="rcl" library_urn="urn:adsk.eagle:library:334" deviceset="R-EU_" device="0204/2V" package3d_urn="urn:adsk.eagle:package:23495/1"/>
-<part name="R6" library="rcl" library_urn="urn:adsk.eagle:library:334" deviceset="R-EU_" device="0204/2V" package3d_urn="urn:adsk.eagle:package:23495/1"/>
-<part name="R7" library="rcl" library_urn="urn:adsk.eagle:library:334" deviceset="R-EU_" device="0204/2V" package3d_urn="urn:adsk.eagle:package:23495/1"/>
-<part name="R8" library="rcl" library_urn="urn:adsk.eagle:library:334" deviceset="R-EU_" device="0204/2V" package3d_urn="urn:adsk.eagle:package:23495/1"/>
-<part name="R9" library="rcl" library_urn="urn:adsk.eagle:library:334" deviceset="R-EU_" device="0204/2V" package3d_urn="urn:adsk.eagle:package:23495/1"/>
-<part name="T2" library="transistor" library_urn="urn:adsk.eagle:library:402" deviceset="2N2222" device="" package3d_urn="urn:adsk.eagle:package:28526/2"/>
-<part name="R10" library="rcl" library_urn="urn:adsk.eagle:library:334" deviceset="R-EU_" device="0204/2V" package3d_urn="urn:adsk.eagle:package:23495/1"/>
+<part name="LED1" library="led" deviceset="LED" device="5MM"/>
+<part name="R1" library="rcl" deviceset="R-EU_" device="0207/7"/>
+<part name="T1" library="transistor" deviceset="2N2222" device=""/>
+<part name="DIS1" library="display-hp" deviceset="HD-H103" device=""/>
+<part name="DIS2" library="display-hp" deviceset="HD-H103" device=""/>
+<part name="IC1" library="ic-package" deviceset="DIL16" device=""/>
+<part name="LED2" library="led" deviceset="LED" device="5MM"/>
+<part name="R2" library="rcl" deviceset="R-EU_" device="0207/7"/>
+<part name="R3" library="rcl" deviceset="R-EU_" device="0207/7"/>
+<part name="R4" library="rcl" deviceset="R-EU_" device="0207/7"/>
+<part name="R5" library="rcl" deviceset="R-EU_" device="0207/7"/>
+<part name="R6" library="rcl" deviceset="R-EU_" device="0207/7"/>
+<part name="R7" library="rcl" deviceset="R-EU_" device="0207/7"/>
+<part name="R8" library="rcl" deviceset="R-EU_" device="0207/7"/>
+<part name="R9" library="rcl" deviceset="R-EU_" device="0207/7"/>
+<part name="T2" library="transistor" deviceset="2N2222" device=""/>
+<part name="R10" library="rcl" deviceset="R-EU_" device="0207/7"/>
+<part name="R11" library="rcl" deviceset="R-EU_" device="0207/7"/>
+<part name="R12" library="rcl" deviceset="R-EU_" device="0207/7"/>
+<part name="R13" library="rcl" deviceset="R-EU_" device="0207/7"/>
+<part name="R14" library="rcl" deviceset="R-EU_" device="0207/7"/>
 </parts>
 <sheets>
@@
 <attribute name="NAME" x="130.81" y="31.9786" size="1.778" layer="95"/>
 <attribute name="VALUE" x="130.81" y="27.178" size="1.778" layer="96"/>
+</instance>
+<instance part="R11" gate="G$1" x="106.68" y="22.86" smashed="yes">
+<attribute name="NAME" x="102.87" y="24.3586" size="1.778" layer="95"/>
+<attribute name="VALUE" x="102.87" y="19.558" size="1.778" layer="96"/>
+</instance>
+<instance part="R12" gate="G$1" x="106.68" y="12.7" smashed="yes">
+<attribute name="NAME" x="102.87" y="14.1986" size="1.778" layer="95"/>
+<attribute name="VALUE" x="102.87" y="9.398" size="1.778" layer="96"/>
+</instance>
+<instance part="R13" gate="G$1" x="134.62" y="73.66" smashed="yes">
+<attribute name="NAME" x="130.81" y="75.1586" size="1.778" layer="95"/>
+<attribute name="VALUE" x="130.81" y="70.358" size="1.778" layer="96"/>
+</instance>
+<instance part="R14" gate="G$1" x="147.32" y="73.66" smashed="yes">
+<attribute name="NAME" x="143.51" y="75.1586" size="1.778" layer="95"/>
+<attribute name="VALUE" x="143.51" y="70.358" size="1.778" layer="96"/>
 </instance>
 </instances>
@@
 </segment>
 </net>
-<net name="N$22" class="0">
-<segment>
-<pinref part="U$1" gate="G$1" pin="31"/>
-<wire x1="96.52" y1="60.96" x2="106.68" y2="60.96" width="0.1524" layer="91"/>
-<wire x1="106.68" y1="60.96" x2="106.68" y2="68.58" width="0.1524" layer="91"/>
-<pinref part="JP1" gate="A" pin="3"/>
-<wire x1="106.68" y1="68.58" x2="119.38" y2="68.58" width="0.1524" layer="91"/>
-</segment>
-</net>
 <net name="N$23" class="0">
 <segment>
 <pinref part="U$1" gate="G$1" pin="33"/>
 <pinref part="JP1" gate="A" pin="4"/>
-<wire x1="96.52" y1="66.04" x2="119.38" y2="66.04" width="0.1524" layer="91"/>
+<wire x1="96.52" y1="66.04" x2="106.68" y2="66.04" width="0.1524" layer="91"/>
+<pinref part="R14" gate="G$1" pin="2"/>
+<wire x1="106.68" y1="66.04" x2="119.38" y2="66.04" width="0.1524" layer="91"/>
+<wire x1="152.4" y1="73.66" x2="152.4" y2="66.04" width="0.1524" layer="91"/>
+<wire x1="152.4" y1="66.04" x2="119.38" y2="66.04" width="0.1524" layer="91"/>
 </segment>
 </net>
@@
 <net name="N$30" class="0">
 <segment>
-<pinref part="T1" gate="G$1" pin="B"/>
-<wire x1="119.38" y1="22.86" x2="96.52" y2="22.86" width="0.1524" layer="91"/>
 <pinref part="U$1" gate="G$1" pin="21"/>
 <wire x1="96.52" y1="22.86" x2="96.52" y2="35.56" width="0.1524" layer="91"/>
+<wire x1="101.6" y1="22.86" x2="96.52" y2="22.86" width="0.1524" layer="91"/>
+<pinref part="R11" gate="G$1" pin="1"/>
 </segment>
 </net>
 <net name="N$28" class="0">
 <segment>
-<pinref part="T2" gate="G$1" pin="B"/>
-<wire x1="119.38" y1="12.7" x2="66.04" y2="12.7" width="0.1524" layer="91"/>
 <pinref part="U$1" gate="G$1" pin="20"/>
 <wire x1="66.04" y1="12.7" x2="66.04" y2="35.56" width="0.1524" layer="91"/>
+<wire x1="101.6" y1="12.7" x2="66.04" y2="12.7" width="0.1524" layer="91"/>
+<pinref part="R12" gate="G$1" pin="1"/>
 </segment>
 </net>
@@
 </segment>
 </net>
+<net name="N$35" class="0">
+<segment>
+<pinref part="T1" gate="G$1" pin="B"/>
+<wire x1="119.38" y1="22.86" x2="111.76" y2="22.86" width="0.1524" layer="91"/>
+<pinref part="R11" gate="G$1" pin="2"/>
+</segment>
+</net>
+<net name="N$36" class="0">
+<segment>
+<pinref part="T2" gate="G$1" pin="B"/>
+<wire x1="119.38" y1="12.7" x2="111.76" y2="12.7" width="0.1524" layer="91"/>
+<pinref part="R12" gate="G$1" pin="2"/>
+</segment>
+</net>
+<net name="N$37" class="0">
+<segment>
+<pinref part="R13" gate="G$1" pin="2"/>
+<pinref part="R14" gate="G$1" pin="1"/>
+<wire x1="139.7" y1="73.66" x2="142.24" y2="73.66" width="0.1524" layer="91"/>
+<pinref part="U$1" gate="G$1" pin="31"/>
+<wire x1="96.52" y1="60.96" x2="139.7" y2="60.96" width="0.1524" layer="91"/>
+<wire x1="139.7" y1="60.96" x2="139.7" y2="73.66" width="0.1524" layer="91"/>
+<junction x="139.7" y="73.66"/>
+</segment>
+</net>
+<net name="N$22" class="0">
+<segment>
+<pinref part="JP1" gate="A" pin="3"/>
+<pinref part="R13" gate="G$1" pin="1"/>
+<wire x1="119.38" y1="68.58" x2="129.54" y2="68.58" width="0.1524" layer="91"/>
+<wire x1="129.54" y1="68.58" x2="129.54" y2="73.66" width="0.1524" layer="91"/>
+</segment>
+</net>
 </nets>
 </sheet>
@@
 </schematic>
 </drawing>
-<compatibility>
-<note version="8.2" severity="warning">
-Since Version 8.2, EAGLE supports online libraries. The ids
-of those online libraries will not be understood (or retained)
-with this version.
-</note>
-<note version="8.3" severity="warning">
-Since Version 8.3, EAGLE supports URNs for individual library
-assets (packages, symbols, and devices). The URNs of those assets
-will not be understood (or retained) with this version.
-</note>
-<note version="8.3" severity="warning">
-Since Version 8.3, EAGLE supports the association of 3D packages
-with devices in libraries, schematics, and board files. Those 3D
-packages will not be understood (or retained) with this version.
-</note>
-<note version="8.4" severity="warning">
-Since Version 8.4, EAGLE supports properties for SPICE simulation.
-Probes in schematics and SPICE mapping objects found in parts and library devices
-will not be understood with this version. Update EAGLE to the latest version
-for full support of SPICE simulation.
-</note>
-</compatibility>
 </eagle>
